File: USB-3-2-splitter/USB-3-2-splitter.kicad_sch (KiCad schematic)
At the start: 35 parts, among them J1 USB_C_Receptacle_USB2.0_16P, J2 USB_C_Receptacle, J3 USB_C_Receptacle, Q1 IRLML6401, Q2 IRLML6401, Q3 IRLML6401, Q4 IRLML6401, U3 SRV05-4

Commit message: Manufacturing files
Parts:
- F1: value 1812L150MR -> 1812L110PR
Changed lines of the file:
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@@
 			)
 		)
-		(property "Value" "1812L150MR"
+		(property "Value" "1812L110PR"
 			(at 72.39 26.4414 90)
 			(effects
