File: USB-3-2-splitter/USB-3-2-splitter.kicad_pcb (KiCad board)
At the start: 4 copper layers, 41 x 29 mm, 35 parts, among them J1 USB_C_Receptacle_USB2.0_16P, J2 USB_C_Receptacle, J3 USB_C_Receptacle, Q1 IRLML6401, Q2 IRLML6401, Q3 IRLML6401, Q4 IRLML6401, U3 SRV05-4

Commit message: Ran DRC
Parts:
- moved H7 0.50 mm to (26.0, 27.5)
Routing:
- net GND: vias 15 -> 20
Other:
- board text added: "JLCJLCJLCJLC"
- board text added: "This takes a USB 3 input (J2) and breaks out the USB2 lines to J1 and the USB3-only lines to J3"
- board text added: "USB-3-2 splitter Pylon April 13, 2025"
- board text added: "USB2"
- board text added: "USB3"
Changed lines of the file:
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@@
 		(tags "USB C Type-C Receptacle SMD")
 		(property "Reference" "J3"
-			(at 0 -6.36 0)
+			(at -6.72 3.34639 0)
 			(layer "F.SilkS")
 			(effects
@@
 	(footprint "USB-3-2-splitter-libraries:JLCPCB-tooling-hole"
 		(layer "F.Cu")
-		(at 26 27)
+		(at 26 27.5)
 		(property "Reference" "H7"
 			(at 0 -2 0)
@@
 		(property "Reference" "H2"
 			(at 0 -3.85 0)
-			(layer "Edge.Cuts")
+			(layer "Eco1.User")
 			(effects
 				(font
@@
 		(tags "usb usb-c 2.0 pd")
 		(property "Reference" "J1"
-			(at -6.22 1.44639 90)
+			(at 5.78 1.34639 90)
 			(layer "F.SilkS")
 			(effects
@@
 		(layer "Edge.Cuts")
 	)
+	(gr_text "USB2"
+		(at 24 26.5 0)
+		(layer "F.SilkS")
+		(effects
+			(font
+				(size 1.2 1.2)
+				(thickness 0.2)
+				(bold yes)
+			)
+			(justify left bottom)
+		)
+	)
+	(gr_text "USB3"
+		(at 19 28.5 0)
+		(layer "F.SilkS")
+		(effects
+			(font
+				(size 1.2 1.2)
+				(thickness 0.2)
+				(bold yes)
+			)
+			(justify left bottom)
+		)
+	)
+	(gr_text "JLCJLCJLCJLC"
+		(at 24.5 4.5 0)
+		(layer "B.SilkS")
+		(effects
+			(font
+				(size 1.2 1.2)
+				(thickness 0.2)
+				(bold yes)
+			)
+			(justify left bottom mirror)
+		)
+	)
+	(gr_text "This takes a USB 3 input (J2) and\nbreaks out the USB2 lines to J1\nand the USB3-only lines to J3"
+		(at 36 20.5 0)
+		(layer "B.SilkS")
+		(effects
+			(font
+				(size 1.2 1.2)
+				(thickness 0.2)
+				(bold yes)
+			)
+			(justify left bottom mirror)
+		)
+	)
+	(gr_text "USB-3-2 splitter\nPylon April 13, 2025\n"
+		(at 31 14 0)
+		(layer "B.SilkS")
+		(effects
+			(font
+				(size 1.5 1.5)
+				(thickness 0.3)
+				(bold yes)
+			)
+			(justify left bottom mirror)
+		)
+	)
 	(segment
 		(start 22.95 26.1375)
@@
 	)
 	(via
+		(at 6.5 12.5)
+		(size 0.6)
+		(drill 0.3)
+		(layers "F.Cu" "B.Cu")
+		(free yes)
+		(net 2)
+	)
+	(via
 		(at 14.1 22.049219)
 		(size 0.4)
@@
 	)
 	(via
+		(at 28 27.5)
+		(size 0.8)
+		(drill 0.4)
+		(layers "F.Cu" "B.Cu")
+		(free yes)
+		(net 2)
+	)
+	(via
+		(at 18 9.5)
+		(size 0.6)
+		(drill 0.3)
+		(layers "F.Cu" "B.Cu")
+		(free yes)
+		(net 2)
+	)
+	(via
 		(at 12.9 10.4)
 		(size 0.6)
@@
 	)
 	(via
+		(at 1.5 16.5)
+		(size 0.8)
+		(drill 0.4)
+		(layers "F.Cu" "B.Cu")
+		(free yes)
+		(net 2)
+	)
+	(via
 		(at 12.9 15.6)
 		(size 0.8)
@@
 		(layers "F.Cu" "B.Cu")
 		(free yes)
+		(net 2)
+	)
+	(via
+		(at 37.5 14.5)
+		(size 0.8)
+		(drill 0.4)
+		(layers "F.Cu" "B.Cu")
+		(free yes)

Commit message: More adjustments
Routing:
- net CC2_USB3: track 37.8 -> 39.3 mm
- net CC1_USB3: track 33.7 -> 34.3 mm
